Commit message: Created core URDF

File: description/robot_core.xacro (robot description, xacro)
@@ -14,4 +14,5 @@
         <color rgba = "0 0 0 1"/>
     </material>
+    <!-- BASE LINK -->
     <link name = "base_link">
     </link>
@@ -40,4 +41,7 @@
         </xacro:inertial_box>
     </link>
+    <gazebo reference="chassis">
+        <material>Gazebo/White</material>
+    </gazebo>
     <!-- LEFT WHEEL LINK -->
     <joint name = "left_wheel_joint" type = "continuous">
@@ -63,4 +67,7 @@
         </xacro:inertial_cylinder>
     </link>
+    <gazebo reference="left_wheel">
+        <material>Gazebo/Blue</material>
+    </gazebo>
     <!-- RIGHT WHEEL LINK -->
     <joint name = "right_wheel_joint" type = "continuous">
@@ -68,5 +75,5 @@
         <child link = "right_wheel"/>
         <origin xyz = "0 -0.175 0" rpy = "${pi/2} 0 0"/>
-        <axis xyz = "0 0 -1"/>
+        <axis xyz = "0 0 1"/>
     </joint>
     <link name = "right_wheel">
@@ -77,13 +84,16 @@
             <material name = "blue"/>
         </visual>
-        <collsion>
+        <collision>
             <geometry>
                 <cylinder radius = "0.05" length = "0.04"/>
             </geometry>
-        </collsion>
+        </collision>
         <xacro:inertial_cylinder mass="0.1" length="0.04" radius="0.05">
             <origin xyz="0 0 0" rpy="0 0 0"/>
         </xacro:inertial_cylinder>
     </link>
+    <gazebo reference="right_wheel">
+        <material>Gazebo/Blue</material>
+    </gazebo>
     <!-- CASTER WHEEL LINK -->
     <joint name = "caster_wheel_joint" type = "fixed">
@@ -108,3 +118,8 @@
         </xacro:inertial_sphere>
     </link>
+    <gazebo reference="caster_wheel">
+        <material>Gazebo/Black</material>
+        <mu1 value="0.001"/>
+        <mu2 value="0.001"/>
+    </gazebo>
 </robot>
